Commit message: Edited sensor frame ids in sdf, added all of the sensor joints into the urdf, all the sensors work and publish properly

File: urdf/ugv.urdf (robot description, URDF)
Before this commit: robot ugv, 40 links, 39 joints
Links:
- added link ugv/camera_back_link/camera_back
- added link ugv/camera_front_link/camera_front
- added link ugv/gps_link/gps
- added link ugv/imu0_link/imu0_sensor
- added link ugv/imu1_link/imu1_sensor
- added link ugv/imu2_link/imu2_sensor
- added link ugv/lidar_2d_link/lidar_2d
- added link ugv/tof_link/tof_range
Joints:
- added joint camera_back_joint: type fixed, parent 360Cam_v4_1, child ugv/camera_back_link/camera_back, origin xyz=-0.022 0 0.093445 rpy=0 0 3.14159
- added joint camera_front_joint: type fixed, parent 360Cam_v4_1, child ugv/camera_front_link/camera_front, origin xyz=0.022 0 0.093445 rpy=0 0 0
- added joint gps_joint: type fixed, parent GPS_v1_1, child ugv/gps_link/gps, origin xyz=0 0.00995 0 rpy=0 0 0
- added joint imu0_joint: type fixed, parent CubeFC_v1_1, child ugv/imu0_link/imu0_sensor, origin xyz=0 0 0 rpy=0 0 0
- added joint imu1_joint: type fixed, parent CubeFC_v1_1, child ugv/imu1_link/imu1_sensor, origin xyz=0 0 0 rpy=0 0 0
- added joint imu2_joint: type fixed, parent CubeFC_v1_1, child ugv/imu2_link/imu2_sensor, origin xyz=0 0 0 rpy=0 0 0
- added joint lidar_2d_joint: type fixed, parent RPLidarC1_v1_1, child ugv/lidar_2d_link/lidar_2d, origin xyz=-0.02780 0 0.03310 rpy=0 0 0
- added joint tof_joint: type fixed, parent TOFSensor_v3_1, child ugv/tof_link/tof_range, origin xyz=0 0 0 rpy=0 0 3.14159

Commit message: Fixed URDF and SDF joints for ackermann drive with cmd_vel

File: urdf/ugv.urdf (robot description, URDF)
Before this commit: robot ugv, 48 links, 47 joints
Joints:
- joint back_right_wheel: axis 0.0 -1.0 0.0 -> 0.0 1.0 0.0
- joint front_right_wheel: axis 0.0 -1.0 0.0 -> 0.0 1.0 0.0
- joint left_steering: axis -0.020219 0.0 -0.999796 -> 0.0 0.0 1.0
- joint right_steering: axis -0.020219 0.0 -0.999796 -> 0.0 0.0 1.0

Commit message: Made wheel collision model into simple cylineders

File: urdf/ugv.urdf (robot description, URDF)
Before this commit: robot ugv, 48 links, 47 joints
Links:
- link BackLeft_1: geometry collision cylinder length=0.050 radius=0.070; visual mesh filename=file:///home/odinroast/Desktop/ros2_ws/install/ugv_descript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 scale=0.001 0.001 0.001
- link BackRight_1: geometry collision cylinder length=0.050 radius=0.070; visual mesh filename=file:///home/odinroast/Desktop/ros2_ws/install/ugv_descript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 scale=0.001 0.001 0.001
- link FrontLeft_1: geometry collision cylinder length=0.050 radius=0.070; visual mesh filename=file:///home/odinroast/Desktop/ros2_ws/install/ugv_descript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 scale=0.001 0.001 0.001
- link FrontRight_1: geometry collision cylinder length=0.050 radius=0.070; visual mesh filename=file:///home/odinroast/Desktop/ros2_ws/install/ugv_descript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 scale=0.001 0.001 0.001

Commit message: Made mass more distributed evenly for 9kg and edited steering joints to be +-45 degrees from +-30 degrees

File: urdf/ugv.urdf (robot description, URDF)
Before this commit: robot ugv, 48 links, 47 joints
Links:
- link BackLeft_1: mass 0.7033756911731642 -> 0.1
- link BackRight_1: mass 0.7033995559753448 -> 0.1
- link FrontLeft_1: mass 0.7033756911731642 -> 0.1
- link FrontRight_1: mass 0.7033995559753448 -> 0.1
- link base_link: mass 0.2720807790827568 -> 8.5
Joints:
- joint left_steering: limit (none) -> lower=-0.7854 upper=0.7854 effort=10 velocity=2.0; type continuous -> revolute
- joint right_steering: limit (none) -> lower=-0.7854 upper=0.7854 effort=10 velocity=2.0; type continuous -> revolute

Commit message: Replaced the path with LIDC path

File: urdf/ugv.urdf (robot description, URDF)
Before this commit: robot ugv, 48 links, 47 joints
Links:
- link 360Cam_v4_1: geometry collision mesh filename=file:///home/lidc/ros2_ws/install/ugv_description/share/ugv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 scale=0.001 0.001 0.001; visual mesh filename=file:///home/lidc/ros2_ws/install/ugv_description/share/ugv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 scale=0.001 0.001 0.001
- link 3ButtonMount_v1_1: geometry collision mesh filename=file:///home/lidc/ros2_ws/install/ugv_description/share/ugv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 scale=0.001 0.001 0.001; visual mesh filename=file:///home/lidc/ros2_ws/install/ugv_description/share/ugv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 scale=0.001 0.001 0.001
- link Anker_737_Power_Bank_v2_1: geometry collision mesh filename=file:///home/lidc/ros2_ws/install/ugv_description/share/ugv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 scale=0.001 0.001 0.001; visual mesh filename=file:///home/lidc/ros2_ws/install/ugv_description/share/ugv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 scale=0.001 0.001 0.001
- link BackLeft_1: geometry collision cylinder length=0.050 radius=0.070; visual mesh filename=file:///home/lidc/ros2_ws/install/ugv_description/share/ugv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 scale=0.001 0.001 0.001
- link BackRight_1: geometry collision cylinder length=0.050 radius=0.070; visual mesh filename=file:///home/lidc/ros2_ws/install/ugv_description/share/ugv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 scale=0.001 0.001 0.001
- link Chassis_1: geometry collision mesh filename=file:///home/lidc/ros2_ws/install/ugv_description/share/ugv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 scale=0.001 0.001 0.001; visual mesh filename=file:///home/lidc/ros2_ws/install/ugv_description/share/ugv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 scale=0.001 0.001 0.001
- link CubeFC_v1_1: geometry collision mesh filename=file:///home/lidc/ros2_ws/install/ugv_description/share/ugv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 scale=0.001 0.001 0.001; visual mesh filename=file:///home/lidc/ros2_ws/install/ugv_description/share/ugv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 scale=0.001 0.001 0.001
- link FrontCover_v1_1: geometry collision mesh filename=file:///home/lidc/ros2_ws/install/ugv_description/share/ugv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 scale=0.001 0.001 0.001; visual mesh filename=file:///home/lidc/ros2_ws/install/ugv_description/share/ugv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 scale=0.001 0.001 0.001
- link FrontLeft_1: geometry collision cylinder length=0.050 radius=0.070; visual mesh filename=file:///home/lidc/ros2_ws/install/ugv_description/share/ugv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 scale=0.001 0.001 0.001
- link FrontLight_v1_1: geometry collision mesh filename=file:///home/lidc/ros2_ws/install/ugv_description/share/ugv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 scale=0.001 0.001 0.001; visual mesh filename=file:///home/lidc/ros2_ws/install/ugv_description/share/ugv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 scale=0.001 0.001 0.001
- link FrontLight_v1__1__1: geometry collision mesh filename=file:///home/lidc/ros2_ws/install/ugv_description/share/ugv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 scale=0.001 0.001 0.001; visual mesh filename=file:///home/lidc/ros2_ws/install/ugv_description/share/ugv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 scale=0.001 0.001 0.001
- link FrontMountFull_v1_1: geometry collision mesh filename=file:///home/lidc/ros2_ws/install/ugv_description/share/ugv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 scale=0.001 0.001 0.001; visual mesh filename=file:///home/lidc/ros2_ws/install/ugv_description/share/ugv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 scale=0.001 0.001 0.001
- link FrontRight_1: geometry collision cylinder length=0.050 radius=0.070; visual mesh filename=file:///home/lidc/ros2_ws/install/ugv_description/share/ugv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 scale=0.001 0.001 0.001
- link GPSMount__1__v1_1: geometry collision mesh filename=file:///home/lidc/ros2_ws/install/ugv_description/share/ugv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 scale=0.001 0.001 0.001; visual mesh filename=file:///home/lidc/ros2_ws/install/ugv_description/share/ugv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 scale=0.001 0.001 0.001
- link GPS_v1_1: geometry collision mesh filename=file:///home/lidc/ros2_ws/install/ugv_description/share/ugv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 scale=0.001 0.001 0.001; visual mesh filename=file:///home/lidc/ros2_ws/install/ugv_description/share/ugv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 scale=0.001 0.001 0.001
- link Insta360MountwithLidar_v1_1: geometry collision mesh filename=file:///home/lidc/ros2_ws/install/ugv_description/share/ugv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 scale=0.001 0.001 0.001; visual mesh filename=file:///home/lidc/ros2_ws/install/ugv_description/share/ugv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 scale=0.001 0.001 0.001
- link JetsonCaseBottom_v1_1: geometry collision mesh filename=file:///home/lidc/ros2_ws/install/ugv_description/share/ugv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 scale=0.001 0.001 0.001; visual mesh filename=file:///home/lidc/ros2_ws/install/ugv_description/share/ugv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 scale=0.001 0.001 0.001
- link JetsonCaseTop_v1_1: geometry collision mesh filename=file:///home/lidc/ros2_ws/install/ugv_description/share/ugv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 scale=0.001 0.001 0.001; visual mesh filename=file:///home/lidc/ros2_ws/install/ugv_description/share/ugv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 scale=0.001 0.001 0.001
- link Jetson_Nano_v1_1: geometry collision mesh filename=file:///home/lidc/ros2_ws/install/ugv_description/share/ugv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 scale=0.001 0.001 0.001; visual mesh filename=file:///home/lidc/ros2_ws/install/ugv_description/share/ugv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 scale=0.001 0.001 0.001
- link KeyHolders_v3_v1_1: geometry collision mesh filename=file:///home/lidc/ros2_ws/install/ugv_description/share/ugv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 scale=0.001 0.001 0.001; visual mesh filename=file:///home/lidc/ros2_ws/install/ugv_description/share/ugv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 scale=0.001 0.001 0.001
- link LIPOBattery_v2_1: geometry collision mesh filename=file:///home/lidc/ros2_ws/install/ugv_description/share/ugv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 scale=0.001 0.001 0.001; visual mesh filename=file:///home/lidc/ros2_ws/install/ugv_description/share/ugv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 scale=0.001 0.001 0.001
- link LeftHub_1: geometry collision mesh filename=file:///home/lidc/ros2_ws/install/ugv_description/share/ugv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 scale=0.001 0.001 0.001; visual mesh filename=file:///home/lidc/ros2_ws/install/ugv_description/share/ugv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 scale=0.001 0.001 0.001
- link LeftSupport_v1_1: geometry collision mesh filename=file:///home/lidc/ros2_ws/install/ugv_description/share/ugv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 scale=0.001 0.001 0.001; visual mesh filename=file:///home/lidc/ros2_ws/install/ugv_description/share/ugv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 scale=0.001 0.001 0.001
- link MountingClipFinal_v1_1: geometry collision mesh filename=file:///home/lidc/ros2_ws/install/ugv_description/share/ugv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 scale=0.001 0.001 0.001; visual mesh filename=file:///home/lidc/ros2_ws/install/ugv_description/share/ugv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 scale=0.001 0.001 0.001
- link MountingClipFinal_v1__1__1: geometry collision mesh filename=file:///home/lidc/ros2_ws/install/ugv_description/share/ugv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 scale=0.001 0.001 0.001; visual mesh filename=file:///home/lidc/ros2_ws/install/ugv_description/share/ugv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 scale=0.001 0.001 0.001
- link MountingClipFinal_v1__2__1: geometry collision mesh filename=file:///home/lidc/ros2_ws/install/ugv_description/share/ugv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 scale=0.001 0.001 0.001; visual mesh filename=file:///home/lidc/ros2_ws/install/ugv_description/share/ugv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 scale=0.001 0.001 0.001
- link MountingClipFinal_v1__3__1: geometry collision mesh filename=file:///home/lidc/ros2_ws/install/ugv_description/share/ugv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 scale=0.001 0.001 0.001; visual mesh filename=file:///home/lidc/ros2_ws/install/ugv_description/share/ugv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 scale=0.001 0.001 0.001
- link Mounting_Plate_v3_v1_1: geometry collision mesh filename=file:///home/lidc/ros2_ws/install/ugv_description/share/ugv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 scale=0.001 0.001 0.001; visual mesh filename=file:///home/lidc/ros2_ws/install/ugv_description/share/ugv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 scale=0.001 0.001 0.001
- link Mounting_Plate_v3_v1__1__1: geometry collision mesh filename=file:///home/lidc/ros2_ws/install/ugv_description/share/ugv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 scale=0.001 0.001 0.001; visual mesh filename=file:///home/lidc/ros2_ws/install/ugv_description/share/ugv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 scale=0.001 0.001 0.001
- link RFD900urdf_v1_1: geometry collision mesh filename=file:///home/lidc/ros2_ws/install/ugv_description/share/ugv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 scale=0.001 0.001 0.001; visual mesh filename=file:///home/lidc/ros2_ws/install/ugv_description/share/ugv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 scale=0.001 0.001 0.001
- link RFDAntenna_v1_1: geometry collision mesh filename=file:///home/lidc/ros2_ws/install/ugv_description/share/ugv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 scale=0.001 0.001 0.001; visual mesh filename=file:///home/lidc/ros2_ws/install/ugv_description/share/ugv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 scale=0.001 0.001 0.001
- link RFDAntenna_v1__1__1: geometry collision mesh filename=file:///home/lidc/ros2_ws/install/ugv_description/share/ugv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 scale=0.001 0.001 0.001; visual mesh filename=file:///home/lidc/ros2_ws/install/ugv_description/share/ugv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 scale=0.001 0.001 0.001
- link RPLidarC1_v1_1: geometry collision mesh filename=file:///home/lidc/ros2_ws/install/ugv_description/share/ugv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 scale=0.001 0.001 0.001; visual mesh filename=file:///home/lidc/ros2_ws/install/ugv_description/share/ugv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 scale=0.001 0.001 0.001
- link RightHub__1: geometry collision mesh filename=file:///home/lidc/ros2_ws/install/ugv_description/share/ugv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 scale=0.001 0.001 0.001; visual mesh filename=file:///home/lidc/ros2_ws/install/ugv_description/share/ugv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 scale=0.001 0.001 0.001
- link RightSupport_v1_1: geometry collision mesh filename=file:///home/lidc/ros2_ws/install/ugv_description/share/ugv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 scale=0.001 0.001 0.001; visual mesh filename=file:///home/lidc/ros2_ws/install/ugv_description/share/ugv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 scale=0.001 0.001 0.001
- link Speaker_v1_1: geometry collision mesh filename=file:///home/lidc/ros2_ws/install/ugv_description/share/ugv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 scale=0.001 0.001 0.001; visual mesh filename=file:///home/lidc/ros2_ws/install/ugv_description/share/ugv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 scale=0.001 0.001 0.001
- link Speaker_v1__1__1: geometry collision mesh filename=file:///home/lidc/ros2_ws/install/ugv_description/share/ugv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 scale=0.001 0.001 0.001; visual mesh filename=file:///home/lidc/ros2_ws/install/ugv_description/share/ugv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 scale=0.001 0.001 0.001
- link TOFSensor_v3_1: geometry collision mesh filename=file:///home/lidc/ros2_ws/install/ugv_description/share/ugv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 scale=0.001 0.001 0.001; visual mesh filename=file:///home/lidc/ros2_ws/install/ugv_description/share/ugv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 scale=0.001 0.001 0.001
- link base_link: geometry collision mesh filename=file:///home/lidc/ros2_ws/install/ugv_description/share/ugv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 scale=0.001 0.001 0.001; visual mesh filename=file:///home/lidc/ros2_ws/install/ugv_description/share/ugv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 scale=0.001 0.001 0.001

Commit message: Fixed IMU orientation in urdf which was not the same as the sdf, this was causing the odomtetry data from the ekf to be interpreted in a false way, also removed the redundant/invalid frame ids from the sdf file to clear warnings clutter when gazebo is launched

File: urdf/ugv.urdf (robot description, URDF)
Before this commit: robot ugv, 48 links, 47 joints
Joints:
- joint imu0_joint: origin xyz=0 0 0 rpy=0 0 0 -> xyz=0 0 0 rpy=3.14159 0 0
- joint imu1_joint: origin xyz=0 0 0 rpy=0 0 0 -> xyz=0 0 0 rpy=3.14159 0 0
- joint imu2_joint: origin xyz=0 0 0 rpy=0 0 0 -> xyz=0 0 0 rpy=3.14159 0 0

Commit message: Simplified all collision meshes in both URDF and SDF to make them much less computationally expensive to run

File: urdf/ugv.urdf (robot description, URDF)
Before this commit: robot ugv, 48 links, 47 joints
Links:
- link 360Cam_v4_1: geometry collision sphere radius=0.03; visual mesh filename=file:///home/odinroast/Desktop/ros2_ws/install/ugv_descript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 scale=0.001 0.001 0.001
- link 3ButtonMount_v1_1: geometry visual mesh filename=file:///home/odinroast/Desktop/ros2_ws/install/ugv_descript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 scale=0.001 0.001 0.001
- link Anker_737_Power_Bank_v2_1: geometry collision box size=0.16 0.08 0.03; visual mesh filename=file:///home/odinroast/Desktop/ros2_ws/install/ugv_descript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 scale=0.001 0.001 0.001
- link Chassis_1: geometry collision box size=0.38 0.28 0.04; visual mesh filename=file:///home/odinroast/Desktop/ros2_ws/install/ugv_descript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 scale=0.001 0.001 0.001
- link CubeFC_v1_1: geometry collision box size=0.04 0.04 0.02; visual mesh filename=file:///home/odinroast/Desktop/ros2_ws/install/ugv_descript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 scale=0.001 0.001 0.001
- link FrontCover_v1_1: geometry collision box size=0.15 0.15 0.003; visual mesh filename=file:///home/odinroast/Desktop/ros2_ws/install/ugv_descript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 scale=0.001 0.001 0.001
- link FrontLight_v1_1: geometry visual mesh filename=file:///home/odinroast/Desktop/ros2_ws/install/ugv_descript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 scale=0.001 0.001 0.001
- link FrontLight_v1__1__1: geometry visual mesh filename=file:///home/odinroast/Desktop/ros2_ws/install/ugv_descript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 scale=0.001 0.001 0.001
- link FrontMountFull_v1_1: geometry collision box size=0.08 0.135 0.02; visual mesh filename=file:///home/odinroast/Desktop/ros2_ws/install/ugv_descript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 scale=0.001 0.001 0.001
- link GPSMount__1__v1_1: geometry visual mesh filename=file:///home/odinroast/Desktop/ros2_ws/install/ugv_descript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 scale=0.001 0.001 0.001
- link GPS_v1_1: geometry collision box size=0.055 0.055 0.015; visual mesh filename=file:///home/odinroast/Desktop/ros2_ws/install/ugv_descript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 scale=0.001 0.001 0.001
- link Insta360MountwithLidar_v1_1: geometry collision box size=0.08 0.06 0.03; visual mesh filename=file:///home/odinroast/Desktop/ros2_ws/install/ugv_descript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 scale=0.001 0.001 0.001
- link JetsonCaseBottom_v1_1: geometry collision box size=0.10 0.06 0.02; visual mesh filename=file:///home/odinroast/Desktop/ros2_ws/install/ugv_descript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 scale=0.001 0.001 0.001
- link JetsonCaseTop_v1_1: geometry visual mesh filename=file:///home/odinroast/Desktop/ros2_ws/install/ugv_descript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 scale=0.001 0.001 0.001
- link Jetson_Nano_v1_1: geometry visual mesh filename=file:///home/odinroast/Desktop/ros2_ws/install/ugv_descript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 scale=0.001 0.001 0.001
- link KeyHolders_v3_v1_1: geometry visual mesh filename=file:///home/odinroast/Desktop/ros2_ws/install/ugv_descript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 scale=0.001 0.001 0.001
- link LIPOBattery_v2_1: geometry collision box size=0.15 0.10 0.04; visual mesh filename=file:///home/odinroast/Desktop/ros2_ws/install/ugv_descript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 scale=0.001 0.001 0.001
- link LeftHub_1: geometry collision cylinder length=0.06 radius=0.03; visual mesh filename=file:///home/odinroast/Desktop/ros2_ws/install/ugv_descript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 scale=0.001 0.001 0.001
- link LeftSupport_v1_1: geometry collision box size=0.20 0.01 0.08; visual mesh filename=file:///home/odinroast/Desktop/ros2_ws/install/ugv_descript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 scale=0.001 0.001 0.001
- link MountingClipFinal_v1_1: geometry visual mesh filename=file:///home/odinroast/Desktop/ros2_ws/install/ugv_descript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 scale=0.001 0.001 0.001
- link MountingClipFinal_v1__1__1: geometry visual mesh filename=file:///home/odinroast/Desktop/ros2_ws/install/ugv_descript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 scale=0.001 0.001 0.001
- link MountingClipFinal_v1__2__1: geometry visual mesh filename=file:///home/odinroast/Desktop/ros2_ws/install/ugv_descript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 scale=0.001 0.001 0.001
- link MountingClipFinal_v1__3__1: geometry visual mesh filename=file:///home/odinroast/Desktop/ros2_ws/install/ugv_descript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 scale=0.001 0.001 0.001
- link Mounting_Plate_v3_v1_1: geometry collision box size=0.27 0.27 0.003; visual mesh filename=file:///home/odinroast/Desktop/ros2_ws/install/ugv_descript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 scale=0.001 0.001 0.001
- link Mounting_Plate_v3_v1__1__1: geometry collision box size=0.27 0.27 0.003; visual mesh filename=file:///home/odinroast/Desktop/ros2_ws/install/ugv_descript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 scale=0.001 0.001 0.001
- link RFD900urdf_v1_1: geometry collision box size=0.06 0.04 0.015; visual mesh filename=file:///home/odinroast/Desktop/ros2_ws/install/ugv_descript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 scale=0.001 0.001 0.001
- link RFDAntenna_v1_1: geometry visual mesh filename=file:///home/odinroast/Desktop/ros2_ws/install/ugv_descript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 scale=0.001 0.001 0.001
- link RFDAntenna_v1__1__1: geometry visual mesh filename=file:///home/odinroast/Desktop/ros2_ws/install/ugv_descript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 scale=0.001 0.001 0.001
- link RPLidarC1_v1_1: geometry collision cylinder length=0.04 radius=0.04; visual mesh filename=file:///home/odinroast/Desktop/ros2_ws/install/ugv_descript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 scale=0.001 0.001 0.001
- link RightHub__1: geometry collision cylinder length=0.06 radius=0.03; visual mesh filename=file:///home/odinroast/Desktop/ros2_ws/install/ugv_descript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 scale=0.001 0.001 0.001
- link RightSupport_v1_1: geometry collision box size=0.20 0.01 0.08; visual mesh filename=file:///home/odinroast/Desktop/ros2_ws/install/ugv_descript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 scale=0.001 0.001 0.001
- link Speaker_v1_1: geometry visual mesh filename=file:///home/odinroast/Desktop/ros2_ws/install/ugv_descript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 scale=0.001 0.001 0.001
- link Speaker_v1__1__1: geometry visual mesh filename=file:///home/odinroast/Desktop/ros2_ws/install/ugv_descript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 scale=0.001 0.001 0.001
- link TOFSensor_v3_1: geometry collision box size=0.02 0.015 0.01; visual mesh filename=file:///home/odinroast/Desktop/ros2_ws/install/ugv_descript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 scale=0.001 0.001 0.001
- link base_link: geometry collision box size=0.40 0.15 0.15; visual mesh filename=file:///home/odinroast/Desktop/ros2_ws/install/ugv_descript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 scale=0.001 0.001 0.001

Commit message: edited urdf and sdf to use basefootprint and then baselink because base footprint is at the center and the ground of the rover, the sdf was changed to make base_footprint into a new frame

File: urdf/ugv.urdf (robot description, URDF)
Before this commit: robot ugv, 48 links, 47 joints
Joints:
- joint base_joint: child base_footprint -> base_link; origin xyz=0.075 -0.075 -0.28375 rpy=0 0 0 -> xyz=-0.075 0.075 0.28375 rpy=0 0 0; parent base_link -> base_footprint
