Commit message: Edited paths to be relative to package

File: urdf/ugv.urdf (robot description, URDF)
Before this commit: robot ugv, 48 links, 47 joints
Links:
- link 360Cam_v4_1: geometry collision sphere radius=0.03; visual mesh filename=package://ugv_description/meshes/360Cam_v4_1.stl scale=0.001 0.001 0.001
- link 3ButtonMount_v1_1: geometry visual mesh filename=package://ugv_description/meshes/3ButtonMount_v1_1.stl scale=0.001 0.001 0.001
- link Anker_737_Power_Bank_v2_1: geometry collision box size=0.16 0.08 0.03; visual mesh filename=package://ugv_description/meshes/Anker_737_Power_Bank_v2_1.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 scale=0.001 0.001 0.001
- link BackLeft_1: geometry collision cylinder length=0.050 radius=0.070; visual mesh filename=package://ugv_description/meshes/BackLeft_1.stl scale=0.001 0.001 0.001
- link BackRight_1: geometry collision cylinder length=0.050 radius=0.070; visual mesh filename=package://ugv_description/meshes/BackRight_1.stl scale=0.001 0.001 0.001
- link Chassis_1: geometry collision box size=0.38 0.28 0.04; visual mesh filename=package://ugv_description/meshes/Chassis_1.stl scale=0.001 0.001 0.001
- link CubeFC_v1_1: geometry collision box size=0.04 0.04 0.02; visual mesh filename=package://ugv_description/meshes/CubeFC_v1_1.stl scale=0.001 0.001 0.001
- link FrontCover_v1_1: geometry collision box size=0.15 0.15 0.003; visual mesh filename=package://ugv_description/meshes/FrontCover_v1_1.stl scale=0.001 0.001 0.001
- link FrontLeft_1: geometry collision cylinder length=0.050 radius=0.070; visual mesh filename=package://ugv_description/meshes/FrontLeft_1.stl scale=0.001 0.001 0.001
- link FrontLight_v1_1: geometry visual mesh filename=package://ugv_description/meshes/FrontLight_v1_1.stl scale=0.001 0.001 0.001
- link FrontLight_v1__1__1: geometry visual mesh filename=package://ugv_description/meshes/FrontLight_v1__1__1.stl scale=0.001 0.001 0.001
- link FrontMountFull_v1_1: geometry collision box size=0.08 0.135 0.02; visual mesh filename=package://ugv_description/meshes/FrontMountFull_v1_1.stl scale=0.001 0.001 0.001
- link FrontRight_1: geometry collision cylinder length=0.050 radius=0.070; visual mesh filename=package://ugv_description/meshes/FrontRight_1.stl scale=0.001 0.001 0.001
- link GPSMount__1__v1_1: geometry visual mesh filename=package://ugv_description/meshes/GPSMount__1__v1_1.stl scale=0.001 0.001 0.001
- link GPS_v1_1: geometry collision box size=0.055 0.055 0.015; visual mesh filename=package://ugv_description/meshes/GPS_v1_1.stl scale=0.001 0.001 0.001
- link Insta360MountwithLidar_v1_1: geometry collision box size=0.08 0.06 0.03; visual mesh filename=package://ugv_description/meshes/Insta360MountwithLidar_v1_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 scale=0.001 0.001 0.001
- link JetsonCaseBottom_v1_1: geometry collision box size=0.10 0.06 0.02; visual mesh filename=package://ugv_description/meshes/JetsonCaseBottom_v1_1.stl scale=0.001 0.001 0.001
- link JetsonCaseTop_v1_1: geometry visual mesh filename=package://ugv_description/meshes/JetsonCaseTop_v1_1.stl scale=0.001 0.001 0.001
- link Jetson_Nano_v1_1: geometry visual mesh filename=package://ugv_description/meshes/Jetson_Nano_v1_1.stl scale=0.001 0.001 0.001
- link KeyHolders_v3_v1_1: geometry visual mesh filename=package://ugv_description/meshes/KeyHolders_v3_v1_1.stl scale=0.001 0.001 0.001
- link LIPOBattery_v2_1: geometry collision box size=0.15 0.10 0.04; visual mesh filename=package://ugv_description/meshes/LIPOBattery_v2_1.stl scale=0.001 0.001 0.001
- link LeftHub_1: geometry collision cylinder length=0.06 radius=0.03; visual mesh filename=package://ugv_description/meshes/LeftHub_1.stl scale=0.001 0.001 0.001
- link LeftSupport_v1_1: geometry collision box size=0.20 0.01 0.08; visual mesh filename=package://ugv_description/meshes/LeftSupport_v1_1.stl scale=0.001 0.001 0.001
- link MountingClipFinal_v1_1: geometry visual mesh filename=package://ugv_description/meshes/MountingClipFinal_v1_1.stl scale=0.001 0.001 0.001
- link MountingClipFinal_v1__1__1: geometry visual mesh filename=package://ugv_description/meshes/MountingClipFinal_v1__1__1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 scale=0.001 0.001 0.001
- link MountingClipFinal_v1__2__1: geometry visual mesh filename=package://ugv_description/meshes/MountingClipFinal_v1__2__1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 scale=0.001 0.001 0.001
- link MountingClipFinal_v1__3__1: geometry visual mesh filename=package://ugv_description/meshes/MountingClipFinal_v1__3__1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 scale=0.001 0.001 0.001
- link Mounting_Plate_v3_v1_1: geometry collision box size=0.27 0.27 0.003; visual mesh filename=package://ugv_description/meshes/Mounting_Plate_v3_v1_1.stl scale=0.001 0.001 0.001
- link Mounting_Plate_v3_v1__1__1: geometry collision box size=0.27 0.27 0.003; visual mesh filename=package://ugv_description/meshes/Mounting_Plate_v3_v1__1__1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 scale=0.001 0.001 0.001
- link RFD900urdf_v1_1: geometry collision box size=0.06 0.04 0.015; visual mesh filename=package://ugv_description/meshes/RFD900urdf_v1_1.stl scale=0.001 0.001 0.001
- link RFDAntenna_v1_1: geometry visual mesh filename=package://ugv_description/meshes/RFDAntenna_v1_1.stl scale=0.001 0.001 0.001
- link RFDAntenna_v1__1__1: geometry visual mesh filename=package://ugv_description/meshes/RFDAntenna_v1__1__1.stl scale=0.001 0.001 0.001
- link RPLidarC1_v1_1: geometry collision cylinder length=0.04 radius=0.04; visual mesh filename=package://ugv_description/meshes/RPLidarC1_v1_1.stl scale=0.001 0.001 0.001
- link RightHub__1: geometry collision cylinder length=0.06 radius=0.03; visual mesh filename=package://ugv_description/meshes/RightHub__1.stl scale=0.001 0.001 0.001
- link RightSupport_v1_1: geometry collision box size=0.20 0.01 0.08; visual mesh filename=package://ugv_description/meshes/RightSupport_v1_1.stl scale=0.001 0.001 0.001
- link Speaker_v1_1: geometry visual mesh filename=package://ugv_description/meshes/Speaker_v1_1.stl scale=0.001 0.001 0.001
- link Speaker_v1__1__1: geometry visual mesh filename=package://ugv_description/meshes/Speaker_v1__1__1.stl scale=0.001 0.001 0.001
- link TOFSensor_v3_1: geometry collision box size=0.02 0.015 0.01; visual mesh filename=package://ugv_description/meshes/TOFSensor_v3_1.stl scale=0.001 0.001 0.001
- link base_link: geometry collision box size=0.40 0.15 0.15; visual mesh filename=package://ugv_description/meshes/base_link.stl scale=0.001 0.001 0.001

Commit message: Edited urdf to flip imu orientations from 180 to zero as cube pilot sends processed imu data already

File: urdf/ugv.urdf (robot description, URDF)
Before this commit: robot ugv, 48 links, 47 joints
Joints:
- joint imu0_joint: origin xyz=0 0 0 rpy=3.14159 0 0 -> xyz=0 0 0 rpy=0 0 0
- joint imu1_joint: origin xyz=0 0 0 rpy=3.14159 0 0 -> xyz=0 0 0 rpy=0 0 0
- joint imu2_joint: origin xyz=0 0 0 rpy=3.14159 0 0 -> xyz=0 0 0 rpy=0 0 0
- joint lidar_2d_joint: origin xyz=-0.02780 0 0.03310 rpy=0 0 0 -> xyz=-0.02780 0 0.03310 rpy=0 0 3.14159
