Commit message: feat: Add comprehensive sensor suite with IMU, lidar, GPS, ToF, and cameras
Add complete sensor integration for UGV simulation with proper URDF link
definitions and Gazebo sensor configurations:

Sensors added:
- IMU sensor (100 Hz, topic: /imu/data)
- 360° RPLidar (30 Hz, 640 samples, 40m range, topic: /lidar)
- VL53L0X ToF range sensor (50 Hz, 0.03-1.0m, topic: /tof/range)
- Here4 GPS/NavSat (10 Hz, 1m accuracy, topic: /gps/fix)
- Insta360 front camera (165° FOV, 640x360@30fps, topic: /camera/front)
- Insta360 back camera (165° FOV, 640x360@30fps, topic: /camera/back)

URDF changes (ugv.xacro):
- Created sensor links with proper inertial properties
- Added fixed joints connecting sensors to physical components
- Positioned sensors with accurate xyz/rpy offsets

Gazebo changes (ugv.gazebo):
- Configured all sensors with realistic parameters
- Added appropriate noise models (GPS, ToF)
- Set up wide-angle camera lens (stereographic projection)
- Configured update rates and topics for each sensor

Documentation:
- Added comprehensive urdf/README.md explaining file structure
- Documented sensor configuration patterns
- Included usage examples and modification guide

File: urdf/ugv.xacro (robot description, xacro)
@@ -151,4 +151,16 @@
   </collision>
 </link>
+<link name="imu_link">
+  <inertial>
+    <mass value="0.001"/>
+    <origin xyz="0 0 0" rpy="0 0 0"/>
+    <inertia ixx="0.0001" ixy="0" ixz="0" iyy="0.0001" iyz="0" izz="0.0001"/>
+  </inertial>
+</link>
+<joint name="imu_joint" type="fixed">
+  <parent link="CubeFC_v1_1"/>  <!-- or base_link -->
+  <child link="imu_link"/>
+  <origin xyz="0 0 0" rpy="0 0 0"/>
+</joint>
 <link name="FrontMountFull_v1_1">
   <inertial>
@@ -511,4 +523,30 @@
   </collision>
 </link>
+<link name="frontcam_link">
+  <inertial>
+    <mass value="0.001"/>
+    <origin xyz="0 0 0" rpy="0 0 0"/>
+    <inertia ixx="0.0001" ixy="0" ixz="0" iyy="0.0001" iyz="0" izz="0.0001"/>
+  </inertial>
+</link>
+<joint name="frontcam_joint" type="fixed">
+  <parent link="360Cam_v4_1"/>
+  <child link="frontcam_link"/>
+  <!-- Offset for camera sensor relative to insta360 camera joint -->
+  <origin xyz="0.022 0 0.093445" rpy="0 0 0"/>
+</joint>
+<link name="backcam_link">
+  <inertial>
+    <mass value="0.001"/>
+    <origin xyz="0 0 0" rpy="0 0 0"/>
+    <inertia ixx="0.0001" ixy="0" ixz="0" iyy="0.0001" iyz="0" izz="0.0001"/>
+  </inertial>
+</link>
+<joint name="backcam_joint" type="fixed">
+  <parent link="360Cam_v4_1"/>
+  <child link="backcam_link"/>
+  <!-- Offset for back camera sensor relative to insta360 camera joint -->
+  <origin xyz="-0.022 0 0.093445" rpy="0 0 3.14159"/>
+</joint>
 <link name="RPLidarC1_v1_1">
   <inertial>
@@ -531,4 +569,17 @@
   </collision>
 </link>
+<link name="360lidar_link">
+  <inertial>
+    <mass value="0.001"/>
+    <origin xyz="0 0 0" rpy="0 0 0"/>
+    <inertia ixx="0.0001" ixy="0" ixz="0" iyy="0.0001" iyz="0" izz="0.0001"/>
+  </inertial>
+</link>
+<joint name="360lidar_joint" type="fixed">
+  <parent link="RPLidarC1_v1_1"/>
+  <child link="360lidar_link"/>
+  <!-- Offset to actual lidar center for gazebo plugin -->
+  <origin xyz="-0.02780 0 0.03310" rpy="0 0 0"/>
+</joint>
 <link name="Chassis_1">
   <inertial>
@@ -631,4 +682,17 @@
   </collision>
 </link>
+<link name="ToFsensor_link">
+  <inertial>
+    <mass value="0.001"/>
+    <origin xyz="0 0 0" rpy="0 0 0"/>
+    <inertia ixx="0.0001" ixy="0" ixz="0" iyy="0.0001" iyz="0" izz="0.0001"/>
+  </inertial>
+</link>
+<joint name="ToFsensor_joint" type="fixed">
+  <parent link="TOFSensor_v3_1"/>
+  <child link="ToFsensor_link"/>
+  <!-- Rotate by 180 so tof sensor looks back -->
+  <origin xyz="0 0 0" rpy="0 0 3.14159"/>
+</joint>
 <link name="LeftHub_1">
   <inertial>
@@ -791,4 +855,17 @@
   </collision>
 </link>
+<link name="GPSsensor_link">
+  <inertial>
+    <mass value="0.001"/>
+    <origin xyz="0 0 0" rpy="0 0 0"/>
+    <inertia ixx="0.0001" ixy="0" ixz="0" iyy="0.0001" iyz="0" izz="0.0001"/>
+  </inertial>
+</link>
+<joint name="GPSsensor_joint" type="fixed">
+  <parent link="GPS_v1_1"/>
+  <child link="GPSsensor_link"/>
+  <!-- Shift the link right so its at the center of the gps -->
+  <origin xyz="0 0.00995 0" rpy="0 0 0"/>
+</joint>
 <joint name="Rigid 2" type="fixed">
   <origin xyz="0.0075 -0.1425 -0.000125" rpy="0 0 0"/>

Commit message: Config folder changes: - Irl and Sim seperate folders, Added gazebo to ros bridge - new file mav.param has default sitl parameters - default display.rviz
Launch folder:
- Edited display.launch.py to launch default params from the sim folder
- added new file for launching rviz, gazebo, and ardupilot sitl together

Urdf folder:
- Accurate files that work

Worlds folder:
- Added iris world so its there locally

setup.py
- Edited to add the new entry point and install config files to the install directory

File: urdf/ugv.xacro (robot description, xacro)
@@ -27,5 +27,5 @@
     <origin xyz="0 0 0" rpy="0 0 0"/>
     <geometry>
-      <mesh filename="file://$(find ugv_description)/meshes/base_link.stl" scale="0.001 0.001 0.001"/>
+      <box size="0.1 0.1 0.1"/>
     </geometry>
   </collision>
@@ -47,5 +47,5 @@
     <origin xyz="-0.0075 0.1425 0.000125" rpy="0 0 0"/>
     <geometry>
-      <mesh filename="file://$(find ugv_description)/meshes/RightSupport_v1_1.stl" scale="0.001 0.001 0.001"/>
+      <box size="0.1 0.1 0.1"/>
     </geometry>
   </collision>
@@ -67,5 +67,5 @@
     <origin xyz="-0.0075 0.0075 0.000125" rpy="0 0 0"/>
     <geometry>
-      <mesh filename="file://$(find ugv_description)/meshes/LeftSupport_v1_1.stl" scale="0.001 0.001 0.001"/>
+      <box size="0.1 0.1 0.1"/>
     </geometry>
   </collision>
@@ -85,7 +85,7 @@
   </visual>
   <collision>
-    <origin xyz="-0.1595 0.1425 0.07325" rpy="0 0 0"/>
-    <geometry>
-      <mesh filename="file://$(find ugv_description)/meshes/Mounting_Plate_v3_v1_1.stl" scale="0.001 0.001 0.001"/>
+    <origin xyz="0 0 0" rpy="0 0 0"/>
+    <geometry>
+      <box size="0.27 0.27 0.003"/>
     </geometry>
   </collision>
@@ -105,7 +105,7 @@
   </visual>
   <collision>
-    <origin xyz="0.0345 0.1425 0.077325" rpy="0 0 0"/>
-    <geometry>
-      <mesh filename="file://$(find ugv_description)/meshes/Mounting_Plate_v3_v1__1__1.stl" scale="0.001 0.001 0.001"/>
+    <origin xyz="0 0 0" rpy="0 0 0"/>
+    <geometry>
+      <box size="0.27 0.27 0.003"/>
     </geometry>
   </collision>
@@ -125,7 +125,7 @@
   </visual>
   <collision>
-    <origin xyz="-0.15 0.075 -0.00145" rpy="0 0 0"/>
-    <geometry>
-      <mesh filename="file://$(find ugv_description)/meshes/FrontCover_v1_1.stl" scale="0.001 0.001 0.001"/>
+    <origin xyz="0 0 0" rpy="0 0 0"/>
+    <geometry>
+      <box size="0.15 0.15 0.003"/>
     </geometry>
   </collision>
@@ -145,7 +145,7 @@
   </visual>
   <collision>
-    <origin xyz="-0.0975 0.1125 0.000125" rpy="0 0 0"/>
-    <geometry>
-      <mesh filename="file://$(find ugv_description)/meshes/CubeFC_v1_1.stl" scale="0.001 0.001 0.001"/>
+    <origin xyz="0 0 0" rpy="0 0 0"/>
+    <geometry>
+      <box size="0.04 0.04 0.02"/>
     </geometry>
   </collision>
@@ -177,7 +177,7 @@
   </visual>
   <collision>
-    <origin xyz="-0.2795 0.0225 0.07325" rpy="0 0 0"/>
-    <geometry>
-      <mesh filename="file://$(find ugv_description)/meshes/FrontMountFull_v1_1.stl" scale="0.001 0.001 0.001"/>
+    <origin xyz="0 0 0" rpy="0 0 0"/>
+    <geometry>
+      <box size="0.08 0.135 0.02"/>
     </geometry>
   </collision>
@@ -199,5 +199,5 @@
     <origin xyz="-0.303776 0.00875 0.072039" rpy="0 0 0"/>
     <geometry>
-      <mesh filename="file://$(find ugv_description)/meshes/FrontLight_v1_1.stl" scale="0.001 0.001 0.001"/>
+      <box size="0.1 0.1 0.1"/>
     </geometry>
   </collision>
@@ -219,5 +219,5 @@
     <origin xyz="-0.303776 0.14375 0.072039" rpy="0 0 0"/>
     <geometry>
-      <mesh filename="file://$(find ugv_description)/meshes/FrontLight_v1__1__1.stl" scale="0.001 0.001 0.001"/>
+      <box size="0.1 0.1 0.1"/>
     </geometry>
   </collision>
@@ -239,5 +239,5 @@
     <origin xyz="-0.305098 0.031776 0.090129" rpy="0 0 0"/>
     <geometry>
-      <mesh filename="file://$(find ugv_description)/meshes/Speaker_v1__1__1.stl" scale="0.001 0.001 0.001"/>
+      <box size="0.1 0.1 0.1"/>
     </geometry>
   </collision>
@@ -259,5 +259,5 @@
     <origin xyz="-0.305098 0.120724 0.090129" rpy="0 0 0"/>
     <geometry>
-      <mesh filename="file://$(find ugv_description)/meshes/Speaker_v1_1.stl" scale="0.001 0.001 0.001"/>
+      <box size="0.1 0.1 0.1"/>
     </geometry>
   </collision>
@@ -277,7 +277,7 @@
   </visual>
   <collision>
-    <origin xyz="0.0945 0.0975 0.077325" rpy="0 0 0"/>
-    <geometry>
-      <mesh filename="file://$(find ugv_description)/meshes/JetsonCaseBottom_v1_1.stl" scale="0.001 0.001 0.001"/>
+    <origin xyz="0 0 0" rpy="0 0 0"/>
+    <geometry>
+      <box size="0.10 0.06 0.02"/>
     </geometry>
   </collision>
@@ -299,5 +299,5 @@
     <origin xyz="0.102 0.0 0.077325" rpy="0 0 0"/>
     <geometry>
-      <mesh filename="file://$(find ugv_description)/meshes/KeyHolders_v3_v1_1.stl" scale="0.001 0.001 0.001"/>
+      <box size="0.1 0.1 0.1"/>
     </geometry>
   </collision>
@@ -319,5 +319,5 @@
     <origin xyz="0.1695 0.0825 0.077325" rpy="0 0 0"/>
     <geometry>
-      <mesh filename="file://$(find ugv_description)/meshes/3ButtonMount_v1_1.stl" scale="0.001 0.001 0.001"/>
+      <box size="0.1 0.1 0.1"/>
     </geometry>
   </collision>
@@ -339,5 +339,5 @@
     <origin xyz="0.354 0.089465 0.157674" rpy="0 0 0"/>
     <geometry>
-      <mesh filename="file://$(find ugv_description)/meshes/RFD900urdf_v1_1.stl" scale="0.001 0.001 0.001"/>
+      <box size="0.1 0.1 0.1"/>
     </geometry>
   </collision>
@@ -359,5 +359,5 @@
     <origin xyz="0.200447 0.085518 0.0864" rpy="0 0 0"/>
     <geometry>
-      <mesh filename="file://$(find ugv_description)/meshes/RFDAntenna_v1__1__1.stl" scale="0.001 0.001 0.001"/>
+      <box size="0.1 0.1 0.1"/>
     </geometry>
   </collision>
@@ -379,5 +379,5 @@
     <origin xyz="0.200447 0.064482 0.0864" rpy="0 0 0"/>
     <geometry>
-      <mesh filename="file://$(find ugv_description)/meshes/RFDAntenna_v1_1.stl" scale="0.001 0.001 0.001"/>
+      <box size="0.1 0.1 0.1"/>
     </geometry>
   </collision>
@@ -399,5 +399,5 @@
     <origin xyz="-0.2795 0.0075 0.07325" rpy="0 0 0"/>
     <geometry>
-      <mesh filename="file://$(find ugv_description)/meshes/MountingClipFinal_v1_1.stl" scale="0.001 0.001 0.001"/>
+      <box size="0.1 0.1 0.1"/>
     </geometry>
   </collision>
@@ -419,5 +419,5 @@
     <origin xyz="-0.2795 0.1425 0.07325" rpy="0 0 0"/>
     <geometry>
-      <mesh filename="file://$(find ugv_description)/meshes/MountingClipFinal_v1__2__1.stl" scale="0.001 0.001 0.001"/>
+      <box size="0.1 0.1 0.1"/>
     </geometry>
   </collision>
@@ -439,5 +439,5 @@
     <origin xyz="0.0795 0.0075 0.0789" rpy="0 0 0"/>
     <geometry>
-      <mesh filename="file://$(find ugv_description)/meshes/MountingClipFinal_v1__1__1.stl" scale="0.001 0.001 0.001"/>
+      <box size="0.1 0.1 0.1"/>
     </geometry>
   </collision>
@@ -459,5 +459,5 @@
     <origin xyz="0.0795 0.1425 0.0789" rpy="0 0 0"/>
     <geometry>
-      <mesh filename="file://$(find ugv_description)/meshes/MountingClipFinal_v1__3__1.stl" scale="0.001 0.001 0.001"/>
+      <box size="0.1 0.1 0.1"/>
     </geometry>
   </collision>
@@ -477,7 +477,7 @@
   </visual>
   <collision>
-    <origin xyz="-0.066 0.075 0.111" rpy="0 0 0"/>
-    <geometry>
-      <mesh filename="file://$(find ugv_description)/meshes/Anker_737_Power_Bank_v2_1.stl" scale="0.001 0.001 0.001"/>
+    <origin xyz="0 0 0.025" rpy="0 0 0"/>
+    <geometry>
+      <box size="0.16 0.08 0.03"/>
     </geometry>
   </collision>
@@ -497,7 +497,7 @@
   </visual>
   <collision>
-    <origin xyz="-0.302 0.075 0.071675" rpy="0 0 0"/>
-    <geometry>
-      <mesh filename="file://$(find ugv_description)/meshes/Insta360MountwithLidar_v1_1.stl" scale="0.001 0.001 0.001"/>
+    <origin xyz="0 0 0" rpy="0 0 0"/>
+    <geometry>
+      <box size="0.08 0.06 0.03"/>
     </geometry>
   </collision>
@@ -517,7 +517,7 @@
   </visual>
   <collision>
-    <origin xyz="-0.1847 0.075 0.050175" rpy="0 0 0"/>
-    <geometry>
-      <mesh filename="file://$(find ugv_description)/meshes/360Cam_v4_1.stl" scale="0.001 0.001 0.001"/>
+    <origin xyz="0 0 0" rpy="0 0 0"/>
+    <geometry>
+      <sphere radius="0.03"/>
     </geometry>
   </collision>
@@ -563,7 +563,7 @@
   </visual>
   <collision>
-    <origin xyz="-0.302 0.075 0.064675" rpy="0 0 0"/>
-    <geometry>
-      <mesh filename="file://$(find ugv_description)/meshes/RPLidarC1_v1_1.stl" scale="0.001 0.001 0.001"/>
+    <origin xyz="0 0 0" rpy="1.5708 0 0"/>
+    <geometry>
+      <cylinder radius="0.04" length="0.04"/>
     </geometry>
   </collision>
@@ -596,7 +596,7 @@
   </visual>
   <collision>
-    <origin xyz="-0.134 0.1475 0.21525" rpy="0 0 0"/>
-    <geometry>
-      <mesh filename="file://$(find ugv_description)/meshes/Chassis_1.stl" scale="0.001 0.001 0.001"/>
+    <origin xyz="-0.05 0.07 0.08" rpy="0 0 0"/>
+    <geometry>
+      <box size="0.38 0.28 0.04"/>
     </geometry>
   </collision>
@@ -618,5 +618,5 @@
     <origin xyz="0.09325 0.096887 0.073325" rpy="0 0 0"/>
     <geometry>
-      <mesh filename="file://$(find ugv_description)/meshes/Jetson_Nano_v1_1.stl" scale="0.001 0.001 0.001"/>
+      <box size="0.1 0.1 0.1"/>
     </geometry>
   </collision>
@@ -638,5 +638,5 @@
     <origin xyz="0.093662 0.039887 0.073325" rpy="0 0 0"/>
     <geometry>
-      <mesh filename="file://$(find ugv_description)/meshes/JetsonCaseTop_v1_1.stl" scale="0.001 0.001 0.001"/>
+      <box size="0.1 0.1 0.1"/>
     </geometry>
   </collision>
@@ -656,7 +656,7 @@
   </visual>
   <collision>
-    <origin xyz="-0.066 0.075 0.135" rpy="0 0 0"/>
-    <geometry>
-      <mesh filename="file://$(find ugv_description)/meshes/LIPOBattery_v2_1.stl" scale="0.001 0.001 0.001"/>
+    <origin xyz="0 0 0.012" rpy="0 0 0"/>
+    <geometry>
+      <box size="0.15 0.10 0.04"/>
     </geometry>
   </collision>
@@ -676,7 +676,7 @@
   </visual>
   <collision>
-    <origin xyz="0.179 0.027743 0.078112" rpy="0 0 0"/>
-    <geometry>
-      <mesh filename="file://$(find ugv_description)/meshes/TOFSensor_v3_1.stl" scale="0.001 0.001 0.001"/>
+    <origin xyz="0 0 0" rpy="0 0 0"/>
+    <geometry>
+      <box size="0.02 0.015 0.01"/>
     </geometry>
   </collision>
@@ -709,7 +709,7 @@
   </visual>
   <collision>
-    <origin xyz="-0.263789 0.004911 0.134519" rpy="0 0 0"/>
-    <geometry>
-      <mesh filename="file://$(find ugv_description)/meshes/LeftHub_1.stl" scale="0.001 0.001 0.001"/>
+    <origin xyz="0 0 -0.04" rpy="1.5708 0 0"/>
+    <geometry>
+      <cylinder radius="0.03" length="0.06"/>
     </geometry>
   </collision>
@@ -729,7 +729,7 @@
   </visual>
   <collision>
-    <origin xyz="-0.263789 0.145089 0.134519" rpy="0 0 0"/>
-    <geometry>
-      <mesh filename="file://$(find ugv_description)/meshes/RightHub__1.stl" scale="0.001 0.001 0.001"/>
+    <origin xyz="0 0 -0.04" rpy="1.5708 0 0"/>
+    <geometry>
+      <cylinder radius="0.03" length="0.06"/>
     </geometry>
   </collision>
@@ -749,7 +749,7 @@
   </visual>
   <collision>
-    <origin xyz="-0.263789 -0.031089 0.213259" rpy="0 0 0"/>
-    <geometry>
-      <mesh filename="file://$(find ugv_description)/meshes/FrontLeft_1.stl" scale="0.001 0.001 0.001"/>
+    <origin xyz="0 0 0" rpy="1.5708 0 0"/>
+    <geometry>
+      <cylinder radius="0.070" length="0.050"/>
     </geometry>
   </collision>
@@ -769,7 +769,7 @@
   </visual>
   <collision>
-    <origin xyz="-0.263789 0.181089 0.213259" rpy="0 0 0"/>
-    <geometry>
-      <mesh filename="file://$(find ugv_description)/meshes/FrontRight_1.stl" scale="0.001 0.001 0.001"/>
+    <origin xyz="0 0 0" rpy="1.5708 0 0"/>
+    <geometry>
+      <cylinder radius="0.070" length="0.050"/>
     </geometry>
   </collision>
@@ -789,7 +789,7 @@
   </visual>
   <collision>
-    <origin xyz="0.071211 -0.031089 0.213259" rpy="0 0 0"/>
-    <geometry>
-      <mesh filename="file://$(find ugv_description)/meshes/BackLeft_1.stl" scale="0.001 0.001 0.001"/>
+    <origin xyz="0 0 0" rpy="1.5708 0 0"/>
+    <geometry>
+      <cylinder radius="0.070" length="0.050"/>
     </geometry>
   </collision>
@@ -809,7 +809,7 @@
   </visual>
   <collision>
-    <origin xyz="0.071211 0.181089 0.213259" rpy="0 0 0"/>
-    <geometry>
-      <mesh filename="file://$(find ugv_description)/meshes/BackRight_1.stl" scale="0.001 0.001 0.001"/>
+    <origin xyz="0 0 0" rpy="1.5708 0 0"/>
+    <geometry>
+      <cylinder radius="0.070" length="0.050"/>
     </geometry>
   </collision>
@@ -831,5 +831,5 @@
     <origin xyz="-0.0075 0.0675 -0.00145" rpy="0 0 0"/>
     <geometry>
-      <mesh filename="file://$(find ugv_description)/meshes/GPSMount__1__v1_1.stl" scale="0.001 0.001 0.001"/>
+      <box size="0.1 0.1 0.1"/>
     </geometry>
   </collision>
@@ -851,5 +851,5 @@
     <origin xyz="0.045886 0.08495 -0.05895" rpy="0 0 0"/>
     <geometry>
-      <mesh filename="file://$(find ugv_description)/meshes/GPS_v1_1.stl" scale="0.001 0.001 0.001"/>
+      <box size="0.1 0.1 0.1"/>
     </geometry>
   </collision>
@@ -1037,5 +1037,5 @@
 </joint>
 <joint name="front_right_wheel" type="continuous">
-  <origin xyz="0.0 -0.036 -0.07874" rpy="0 0 0"/>
+  <origin xyz="0.0 -0.036 -0.07874" rpy="3.14159 0 0"/>
   <parent link="RightHub__1"/>
   <child link="FrontRight_1"/>
@@ -1049,5 +1049,5 @@
 </joint>
 <joint name="back_right_wheel" type="continuous">
-  <origin xyz="-0.205211 -0.033589 0.001991" rpy="0 0 0"/>
+  <origin xyz="-0.205211 -0.033589 0.001991" rpy="3.14159 0 0"/>
   <parent link="Chassis_1"/>
   <child link="BackRight_1"/>

Commit message: feat: integrate Cartographer SLAM with base_footprint frame hierarchy
Major Changes:
- Restructure robot TF tree with base_footprint as root frame instead of base_link
- Add complete Cartographer SLAM integration with ArduPilot external odometry support
- Configure sensor frame mappings for Gazebo's auto-generated frame hierarchy

URDF Changes:
- Invert base_joint: parent=base_footprint, child=base_link
- Update joint transform to xyz=-0.075 0.075 0.28375 (negated from original)
- Maintain IMU correctly mounted on CubeFC_v1_1 (no changes to IMU mount)

Gazebo Configuration:
- Update ArduPilot plugin imuName: base_link::imu_sensor to base_footprint::imu_sensor
- Update odometry plugin robot_base_frame: base_link to base_footprint
- Bridge IMU using full Gazebo sensor path

Cartographer SLAM:
- Add cartographer.launch.py with SLAM nodes and ArduPilot TF relay
- Add cartographer_rover.lua config (2D SLAM, RPLidar 0.15-12m range, IMU enabled)
- Add cartographer_rover.rviz for SLAM visualization
- Configure QoS overrides (reliable) for sensor topics from Gazebo
- Add static TF publishers for IMU and lidar sensor frames
- Add TF relay: /tf to /ap/tf for ArduPilot EKF3 external odometry

Launch Files:
- Update ugv_sitl_gz.launch.py lidar static TF: base_link to base_footprint

Package Setup:
- Add slam/ subdirectory to launch file installation
- Add config/cartographer/ directory installation

Documentation:
- Add comprehensive README.md explaining Cartographer-ArduPilot integration
- Document data flow and troubleshooting guide

Technical Notes:
- IMU static TF uses identity transform (workaround for Cartographer colocation requirement)
- ArduPilot subscribes to /ap/tf expecting odom to base_link transforms
- EKF3 configured with EK3_SRC1_POSXY=3, VELXY=3 for external navigation source

File: urdf/ugv.xacro (robot description, xacro)
@@ -7,7 +7,7 @@
 <link name="base_footprint"/>
 <joint name="base_joint" type="fixed">
-  <parent link="base_link"/>
-  <child link="base_footprint"/>
-  <origin xyz="0.075 -0.075 -0.28375" rpy="0 0 0"/>
+  <parent link="base_footprint"/>
+  <child link="base_link"/>
+  <origin xyz="-0.075 0.075 0.28375" rpy="0 0 0"/>
 </joint>
 <link name="base_link">

Commit message: config: - Edited display.rviz to include laser scan, nav2 plugin and the cartographer map - Edited mav.param to take in external odom and not crash out using internal AHRS odom - Added nav2.params file that uses a basic MPPI controller to move the rover, still need to add collision mointoring and code that will letthe rover turn properly around corners launch: - Added joystick.launch file that launches the ros2_joy package that pubs the joystick data and pubs it as cmd_vel (1:1) mapping as of now - Added navigation.launch file that launches nav2 from the custom parameter file - gz_sitl_launch: Removed uneccessary imports and updated comments ugv_description: - Created the controller node that converts ros2/joy data to cmd_vel
urdf
- xacro: Changed steering joints from continuous to revolute and added joint limits to the steering (+- 45 degrees)
- gazebo: Tuned ardupilot plugin to be more responsive and edited wheels to have friction

setup.py
- added entry point for xbox node

File: urdf/ugv.xacro (robot description, xacro)
@@ -1018,15 +1018,17 @@
   <child link="TOFSensor_v3_1"/>
 </joint>
-<joint name="left_steering" type="continuous">
+<joint name="left_steering" type="revolute">
   <origin xyz="0.129789 0.142589 0.080731" rpy="0 0 0"/>
   <parent link="Chassis_1"/>
   <child link="LeftHub_1"/>
   <axis xyz="-0.020219 0.0 -0.999796"/>
-</joint>
-<joint name="right_steering" type="continuous">
+  <limit lower="-0.785398" upper="0.785398" effort="10" velocity="10"/>
+</joint>
+<joint name="right_steering" type="revolute">
   <origin xyz="0.129789 0.002411 0.080731" rpy="0 0 0"/>
   <parent link="Chassis_1"/>
   <child link="RightHub__1"/>
   <axis xyz="-0.020219 0.0 -0.999796"/>
+  <limit lower="-0.785398" upper="0.785398" effort="10" velocity="10"/>
 </joint>
 <joint name="front_left_wheel" type="continuous">
