Commit message: Edited everything to ensure base_footprint is now base link at the center of the rover and the old base_link is renamed to base_plate, this makes translation into ardupilot stuff much easier

File: urdf/ugv.xacro (robot description, xacro)
@@ -5,11 +5,11 @@
 <xacro:include filename="$(find ugv_description)/urdf/ugv.gazebo" />
 <!-- Robot Footprint -->
-<link name="base_footprint"/>
+<link name="base_link"/>
 <joint name="base_joint" type="fixed">
-  <parent link="base_footprint"/>
-  <child link="base_link"/>
+  <parent link="base_link"/>
+  <child link="base_plate"/>
   <origin xyz="-0.075 0.075 0.28375" rpy="0 0 0"/>
 </joint>
-<link name="base_link">
+<link name="base_plate">
   <inertial>
     <origin xyz="0.07499999999999711 -0.07499999999999997 0.0006625999999999998" rpy="0 0 0"/>
@@ -20,5 +20,5 @@
     <origin xyz="0 0 0" rpy="0 0 0"/>
     <geometry>
-      <mesh filename="file://$(find ugv_description)/meshes/base_link.stl" scale="0.001 0.001 0.001"/>
+      <mesh filename="file://$(find ugv_description)/meshes/base_plate.stl" scale="0.001 0.001 0.001"/>
     </geometry>
     <material name="silver"/>
@@ -159,5 +159,5 @@
 </link>
 <joint name="imu_joint" type="fixed">
-  <parent link="CubeFC_v1_1"/>  <!-- or base_link -->
+  <parent link="CubeFC_v1_1"/>  <!-- or base_plate -->
   <child link="imu_link"/>
   <origin xyz="0 0 0" rpy="0 0 0"/>
@@ -870,10 +870,10 @@
 <joint name="Rigid 2" type="fixed">
   <origin xyz="0.0075 -0.1425 -0.000125" rpy="0 0 0"/>
-  <parent link="base_link"/>
+  <parent link="base_plate"/>
   <child link="RightSupport_v1_1"/>
 </joint>
 <joint name="Rigid 3" type="fixed">
   <origin xyz="0.0075 -0.0075 -0.000125" rpy="0 0 0"/>
-  <parent link="base_link"/>
+  <parent link="base_plate"/>
   <child link="LeftSupport_v1_1"/>
 </joint>
@@ -890,10 +890,10 @@
 <joint name="Rigid 7" type="fixed">
   <origin xyz="0.15 -0.075 0.00145" rpy="0 0 0"/>
-  <parent link="base_link"/>
+  <parent link="base_plate"/>
   <child link="FrontCover_v1_1"/>
 </joint>
 <joint name="Rigid 11" type="fixed">
   <origin xyz="0.0975 -0.1125 -0.000125" rpy="0 0 0"/>
-  <parent link="base_link"/>
+  <parent link="base_plate"/>
   <child link="CubeFC_v1_1"/>
 </joint>
@@ -1058,5 +1058,5 @@
 <joint name="Rigid 58" type="fixed">
   <origin xyz="0.0075 -0.0675 0.00145" rpy="0 0 0"/>
-  <parent link="base_link"/>
+  <parent link="base_plate"/>
   <child link="GPSMount__1__v1_1"/>
 </joint>

Commit message: Redid the urdf to have package relative paths

File: urdf/ugv.xacro (robot description, xacro)
@@ -20,5 +20,5 @@
     <origin xyz="0 0 0" rpy="0 0 0"/>
     <geometry>
-      <mesh filename="file://$(find ugv_description)/meshes/base_plate.stl" scale="0.001 0.001 0.001"/>
+      <mesh filename="package://ugv_description/meshes/base_plate.stl" scale="0.001 0.001 0.001"/>
     </geometry>
     <material name="silver"/>
@@ -40,5 +40,5 @@
     <origin xyz="-0.0075 0.1425 0.000125" rpy="0 0 0"/>
     <geometry>
-      <mesh filename="file://$(find ugv_description)/meshes/RightSupport_v1_1.stl" scale="0.001 0.001 0.001"/>
+      <mesh filename="package://ugv_description/meshes/RightSupport_v1_1.stl" scale="0.001 0.001 0.001"/>
     </geometry>
     <material name="silver"/>
@@ -60,5 +60,5 @@
     <origin xyz="-0.0075 0.0075 0.000125" rpy="0 0 0"/>
     <geometry>
-      <mesh filename="file://$(find ugv_description)/meshes/LeftSupport_v1_1.stl" scale="0.001 0.001 0.001"/>
+      <mesh filename="package://ugv_description/meshes/LeftSupport_v1_1.stl" scale="0.001 0.001 0.001"/>
     </geometry>
     <material name="silver"/>
@@ -80,5 +80,5 @@
     <origin xyz="-0.1595 0.1425 0.07325" rpy="0 0 0"/>
     <geometry>
-      <mesh filename="file://$(find ugv_description)/meshes/Mounting_Plate_v3_v1_1.stl" scale="0.001 0.001 0.001"/>
+      <mesh filename="package://ugv_description/meshes/Mounting_Plate_v3_v1_1.stl" scale="0.001 0.001 0.001"/>
     </geometry>
     <material name="silver"/>
@@ -100,5 +100,5 @@
     <origin xyz="0.0345 0.1425 0.077325" rpy="0 0 0"/>
     <geometry>
-      <mesh filename="file://$(find ugv_description)/meshes/Mounting_Plate_v3_v1__1__1.stl" scale="0.001 0.001 0.001"/>
+      <mesh filename="package://ugv_description/meshes/Mounting_Plate_v3_v1__1__1.stl" scale="0.001 0.001 0.001"/>
     </geometry>
     <material name="silver"/>
@@ -120,5 +120,5 @@
     <origin xyz="-0.15 0.075 -0.00145" rpy="0 0 0"/>
     <geometry>
-      <mesh filename="file://$(find ugv_description)/meshes/FrontCover_v1_1.stl" scale="0.001 0.001 0.001"/>
+      <mesh filename="package://ugv_description/meshes/FrontCover_v1_1.stl" scale="0.001 0.001 0.001"/>
     </geometry>
     <material name="silver"/>
@@ -140,5 +140,5 @@
     <origin xyz="-0.0975 0.1125 0.000125" rpy="0 0 0"/>
     <geometry>
-      <mesh filename="file://$(find ugv_description)/meshes/CubeFC_v1_1.stl" scale="0.001 0.001 0.001"/>
+      <mesh filename="package://ugv_description/meshes/CubeFC_v1_1.stl" scale="0.001 0.001 0.001"/>
     </geometry>
     <material name="silver"/>
@@ -172,5 +172,5 @@
     <origin xyz="-0.2795 0.0225 0.07325" rpy="0 0 0"/>
     <geometry>
-      <mesh filename="file://$(find ugv_description)/meshes/FrontMountFull_v1_1.stl" scale="0.001 0.001 0.001"/>
+      <mesh filename="package://ugv_description/meshes/FrontMountFull_v1_1.stl" scale="0.001 0.001 0.001"/>
     </geometry>
     <material name="silver"/>
@@ -192,5 +192,5 @@
     <origin xyz="-0.303776 0.00875 0.072039" rpy="0 0 0"/>
     <geometry>
-      <mesh filename="file://$(find ugv_description)/meshes/FrontLight_v1_1.stl" scale="0.001 0.001 0.001"/>
+      <mesh filename="package://ugv_description/meshes/FrontLight_v1_1.stl" scale="0.001 0.001 0.001"/>
     </geometry>
     <material name="silver"/>
@@ -212,5 +212,5 @@
     <origin xyz="-0.303776 0.14375 0.072039" rpy="0 0 0"/>
     <geometry>
-      <mesh filename="file://$(find ugv_description)/meshes/FrontLight_v1__1__1.stl" scale="0.001 0.001 0.001"/>
+      <mesh filename="package://ugv_description/meshes/FrontLight_v1__1__1.stl" scale="0.001 0.001 0.001"/>
     </geometry>
     <material name="silver"/>
@@ -232,5 +232,5 @@
     <origin xyz="-0.305098 0.031776 0.090129" rpy="0 0 0"/>
     <geometry>
-      <mesh filename="file://$(find ugv_description)/meshes/Speaker_v1__1__1.stl" scale="0.001 0.001 0.001"/>
+      <mesh filename="package://ugv_description/meshes/Speaker_v1__1__1.stl" scale="0.001 0.001 0.001"/>
     </geometry>
     <material name="silver"/>
@@ -252,5 +252,5 @@
     <origin xyz="-0.305098 0.120724 0.090129" rpy="0 0 0"/>
     <geometry>
-      <mesh filename="file://$(find ugv_description)/meshes/Speaker_v1_1.stl" scale="0.001 0.001 0.001"/>
+      <mesh filename="package://ugv_description/meshes/Speaker_v1_1.stl" scale="0.001 0.001 0.001"/>
     </geometry>
     <material name="silver"/>
@@ -272,5 +272,5 @@
     <origin xyz="0.0945 0.0975 0.077325" rpy="0 0 0"/>
     <geometry>
-      <mesh filename="file://$(find ugv_description)/meshes/JetsonCaseBottom_v1_1.stl" scale="0.001 0.001 0.001"/>
+      <mesh filename="package://ugv_description/meshes/JetsonCaseBottom_v1_1.stl" scale="0.001 0.001 0.001"/>
     </geometry>
     <material name="silver"/>
@@ -292,5 +292,5 @@
     <origin xyz="0.102 0.0 0.077325" rpy="0 0 0"/>
     <geometry>
-      <mesh filename="file://$(find ugv_description)/meshes/KeyHolders_v3_v1_1.stl" scale="0.001 0.001 0.001"/>
+      <mesh filename="package://ugv_description/meshes/KeyHolders_v3_v1_1.stl" scale="0.001 0.001 0.001"/>
     </geometry>
     <material name="silver"/>
@@ -312,5 +312,5 @@
     <origin xyz="0.1695 0.0825 0.077325" rpy="0 0 0"/>
     <geometry>
-      <mesh filename="file://$(find ugv_description)/meshes/3ButtonMount_v1_1.stl" scale="0.001 0.001 0.001"/>
+      <mesh filename="package://ugv_description/meshes/3ButtonMount_v1_1.stl" scale="0.001 0.001 0.001"/>
     </geometry>
     <material name="silver"/>
@@ -332,5 +332,5 @@
     <origin xyz="0.354 0.089465 0.157674" rpy="0 0 0"/>
     <geometry>
-      <mesh filename="file://$(find ugv_description)/meshes/RFD900urdf_v1_1.stl" scale="0.001 0.001 0.001"/>
+      <mesh filename="package://ugv_description/meshes/RFD900urdf_v1_1.stl" scale="0.001 0.001 0.001"/>
     </geometry>
     <material name="silver"/>
@@ -352,5 +352,5 @@
     <origin xyz="0.200447 0.085518 0.0864" rpy="0 0 0"/>
     <geometry>
-      <mesh filename="file://$(find ugv_description)/meshes/RFDAntenna_v1__1__1.stl" scale="0.001 0.001 0.001"/>
+      <mesh filename="package://ugv_description/meshes/RFDAntenna_v1__1__1.stl" scale="0.001 0.001 0.001"/>
     </geometry>
     <material name="silver"/>
@@ -372,5 +372,5 @@
     <origin xyz="0.200447 0.064482 0.0864" rpy="0 0 0"/>
     <geometry>
-      <mesh filename="file://$(find ugv_description)/meshes/RFDAntenna_v1_1.stl" scale="0.001 0.001 0.001"/>
+      <mesh filename="package://ugv_description/meshes/RFDAntenna_v1_1.stl" scale="0.001 0.001 0.001"/>
     </geometry>
     <material name="silver"/>
@@ -392,5 +392,5 @@
     <origin xyz="-0.2795 0.0075 0.07325" rpy="0 0 0"/>
     <geometry>
-      <mesh filename="file://$(find ugv_description)/meshes/MountingClipFinal_v1_1.stl" scale="0.001 0.001 0.001"/>
+      <mesh filename="package://ugv_description/meshes/MountingClipFinal_v1_1.stl" scale="0.001 0.001 0.001"/>
     </geometry>
     <material name="silver"/>
@@ -412,5 +412,5 @@
     <origin xyz="-0.2795 0.1425 0.07325" rpy="0 0 0"/>
     <geometry>
-      <mesh filename="file://$(find ugv_description)/meshes/MountingClipFinal_v1__2__1.stl" scale="0.001 0.001 0.001"/>
+      <mesh filename="package://ugv_description/meshes/MountingClipFinal_v1__2__1.stl" scale="0.001 0.001 0.001"/>
     </geometry>
     <material name="silver"/>
@@ -432,5 +432,5 @@
     <origin xyz="0.0795 0.0075 0.0789" rpy="0 0 0"/>
     <geometry>
-      <mesh filename="file://$(find ugv_description)/meshes/MountingClipFinal_v1__1__1.stl" scale="0.001 0.001 0.001"/>
+      <mesh filename="package://ugv_description/meshes/MountingClipFinal_v1__1__1.stl" scale="0.001 0.001 0.001"/>
     </geometry>
     <material name="silver"/>
@@ -452,5 +452,5 @@
     <origin xyz="0.0795 0.1425 0.0789" rpy="0 0 0"/>
     <geometry>
-      <mesh filename="file://$(find ugv_description)/meshes/MountingClipFinal_v1__3__1.stl" scale="0.001 0.001 0.001"/>
+      <mesh filename="package://ugv_description/meshes/MountingClipFinal_v1__3__1.stl" scale="0.001 0.001 0.001"/>
     </geometry>
     <material name="silver"/>
@@ -472,5 +472,5 @@
     <origin xyz="-0.066 0.075 0.111" rpy="0 0 0"/>
     <geometry>
-      <mesh filename="file://$(find ugv_description)/meshes/Anker_737_Power_Bank_v2_1.stl" scale="0.001 0.001 0.001"/>
+      <mesh filename="package://ugv_description/meshes/Anker_737_Power_Bank_v2_1.stl" scale="0.001 0.001 0.001"/>
     </geometry>
     <material name="silver"/>
@@ -492,5 +492,5 @@
     <origin xyz="-0.302 0.075 0.071675" rpy="0 0 0"/>
     <geometry>
-      <mesh filename="file://$(find ugv_description)/meshes/Insta360MountwithLidar_v1_1.stl" scale="0.001 0.001 0.001"/>
+      <mesh filename="package://ugv_description/meshes/Insta360MountwithLidar_v1_1.stl" scale="0.001 0.001 0.001"/>
     </geometry>
     <material name="silver"/>
@@ -512,5 +512,5 @@
     <origin xyz="-0.1847 0.075 0.050175" rpy="0 0 0"/>
     <geometry>
-      <mesh filename="file://$(find ugv_description)/meshes/360Cam_v4_1.stl" scale="0.001 0.001 0.001"/>
+      <mesh filename="package://ugv_description/meshes/360Cam_v4_1.stl" scale="0.001 0.001 0.001"/>
     </geometry>
     <material name="silver"/>
@@ -558,5 +558,5 @@
     <origin xyz="-0.302 0.075 0.064675" rpy="0 0 0"/>
     <geometry>
-      <mesh filename="file://$(find ugv_description)/meshes/RPLidarC1_v1_1.stl" scale="0.001 0.001 0.001"/>
+      <mesh filename="package://ugv_description/meshes/RPLidarC1_v1_1.stl" scale="0.001 0.001 0.001"/>
     </geometry>
     <material name="silver"/>
@@ -591,5 +591,5 @@
     <origin xyz="-0.134 0.1475 0.21525" rpy="0 0 0"/>
     <geometry>
-      <mesh filename="file://$(find ugv_description)/meshes/Chassis_1.stl" scale="0.001 0.001 0.001"/>
+      <mesh filename="package://ugv_description/meshes/Chassis_1.stl" scale="0.001 0.001 0.001"/>
     </geometry>
     <material name="silver"/>
@@ -611,5 +611,5 @@
     <origin xyz="0.09325 0.096887 0.073325" rpy="0 0 0"/>
     <geometry>
-      <mesh filename="file://$(find ugv_description)/meshes/Jetson_Nano_v1_1.stl" scale="0.001 0.001 0.001"/>
+      <mesh filename="package://ugv_description/meshes/Jetson_Nano_v1_1.stl" scale="0.001 0.001 0.001"/>
     </geometry>
     <material name="silver"/>
@@ -631,5 +631,5 @@
     <origin xyz="0.093662 0.039887 0.073325" rpy="0 0 0"/>
     <geometry>
-      <mesh filename="file://$(find ugv_description)/meshes/JetsonCaseTop_v1_1.stl" scale="0.001 0.001 0.001"/>
+      <mesh filename="package://ugv_description/meshes/JetsonCaseTop_v1_1.stl" scale="0.001 0.001 0.001"/>
     </geometry>
     <material name="silver"/>
@@ -651,5 +651,5 @@
     <origin xyz="-0.066 0.075 0.135" rpy="0 0 0"/>
     <geometry>
-      <mesh filename="file://$(find ugv_description)/meshes/LIPOBattery_v2_1.stl" scale="0.001 0.001 0.001"/>
+      <mesh filename="package://ugv_description/meshes/LIPOBattery_v2_1.stl" scale="0.001 0.001 0.001"/>
     </geometry>
     <material name="silver"/>
@@ -671,5 +671,5 @@
     <origin xyz="0.179 0.027743 0.078112" rpy="0 0 0"/>
     <geometry>
-      <mesh filename="file://$(find ugv_description)/meshes/TOFSensor_v3_1.stl" scale="0.001 0.001 0.001"/>
+      <mesh filename="package://ugv_description/meshes/TOFSensor_v3_1.stl" scale="0.001 0.001 0.001"/>
     </geometry>
     <material name="silver"/>
@@ -704,5 +704,5 @@
     <origin xyz="-0.263789 0.004911 0.134519" rpy="0 0 0"/>
     <geometry>
-      <mesh filename="file://$(find ugv_description)/meshes/LeftHub_1.stl" scale="0.001 0.001 0.001"/>
+      <mesh filename="package://ugv_description/meshes/LeftHub_1.stl" scale="0.001 0.001 0.001"/>
     </geometry>
     <material name="silver"/>
@@ -724,5 +724,5 @@
     <origin xyz="-0.263789 0.145089 0.134519" rpy="0 0 0"/>
     <geometry>
-      <mesh filename="file://$(find ugv_description)/meshes/RightHub__1.stl" scale="0.001 0.001 0.001"/>
+      <mesh filename="package://ugv_description/meshes/RightHub__1.stl" scale="0.001 0.001 0.001"/>
     </geometry>
     <material name="silver"/>
@@ -744,5 +744,5 @@
     <origin xyz="-0.263789 -0.031089 0.213259" rpy="0 0 0"/>
     <geometry>
-      <mesh filename="file://$(find ugv_description)/meshes/FrontLeft_1.stl" scale="0.001 0.001 0.001"/>
+      <mesh filename="package://ugv_description/meshes/FrontLeft_1.stl" scale="0.001 0.001 0.001"/>
     </geometry>
     <material name="silver"/>
@@ -764,5 +764,5 @@
     <origin xyz="-0.263789 0.181089 0.213259" rpy="0 0 0"/>
     <geometry>
-      <mesh filename="file://$(find ugv_description)/meshes/FrontRight_1.stl" scale="0.001 0.001 0.001"/>
+      <mesh filename="package://ugv_description/meshes/FrontRight_1.stl" scale="0.001 0.001 0.001"/>
     </geometry>
     <material name="silver"/>
@@ -784,5 +784,5 @@
     <origin xyz="0.071211 -0.031089 0.213259" rpy="0 0 0"/>
     <geometry>
-      <mesh filename="file://$(find ugv_description)/meshes/BackLeft_1.stl" scale="0.001 0.001 0.001"/>
+      <mesh filename="package://ugv_description/meshes/BackLeft_1.stl" scale="0.001 0.001 0.001"/>
     </geometry>
     <material name="silver"/>
@@ -804,5 +804,5 @@
     <origin xyz="0.071211 0.181089 0.213259" rpy="0 0 0"/>
     <geometry>
-      <mesh filename="file://$(find ugv_description)/meshes/BackRight_1.stl" scale="0.001 0.001 0.001"/>
+      <mesh filename="package://ugv_description/meshes/BackRight_1.stl" scale="0.001 0.001 0.001"/>
     </geometry>
     <material name="silver"/>
@@ -824,5 +824,5 @@
     <origin xyz="-0.0075 0.0675 -0.00145" rpy="0 0 0"/>
     <geometry>
-      <mesh filename="file://$(find ugv_description)/meshes/GPSMount__1__v1_1.stl" scale="0.001 0.001 0.001"/>
+      <mesh filename="package://ugv_description/meshes/GPSMount__1__v1_1.stl" scale="0.001 0.001 0.001"/>
     </geometry>
     <material name="silver"/>
@@ -844,5 +844,5 @@
     <origin xyz="0.045886 0.08495 -0.05895" rpy="0 0 0"/>
     <geometry>
-      <mesh filename="file://$(find ugv_description)/meshes/GPS_v1_1.stl" scale="0.001 0.001 0.001"/>
+      <mesh filename="package://ugv_description/meshes/GPS_v1_1.stl" scale="0.001 0.001 0.001"/>
     </geometry>
     <material name="silver"/>

Commit message: Rotated the lidar link 180 degrees in the urdf and cancelled out that rotation in gazebo because of how the rp lidar c1 treats its LIDAR data

File: urdf/ugv.xacro (robot description, xacro)
@@ -580,5 +580,5 @@
   <child link="360lidar_link"/>
   <!-- Offset to actual lidar center for gazebo plugin -->
-  <origin xyz="-0.02780 0 0.03310" rpy="0 0 0"/>
+  <origin xyz="-0.02780 0 0.03310" rpy="0 0 3.141592653589793"/>
 </joint>
 <link name="Chassis_1">
